Commit message: 修改了几个控制启动脚本,新增参数用于切换v10/v11结构版本;硬件接口文件也适配了不同结构版本的关节限位参数

File: openarm_bimanual_moveit_config/config/openarm_bimanual.urdf.xacro (robot description, xacro)
@@ -13,8 +13,10 @@
 -->
 <robot xmlns:xacro="http://www.ros.org/wiki/xacro" name="openarm_bimanual">
+    <xacro:arg name="arm_type" default="v10" />
     <xacro:arg name="initial_positions_file" default="initial_positions.yaml" />
     <xacro:arg name="hardware_type" default="real" />
+    <xacro:property name="arm_type" value="$(arg arm_type)" />
     <!-- Import openarm_bimanual urdf file -->
-    <xacro:include filename="$(find openarm_description)/urdf/robot/v10.urdf.xacro" />
+    <xacro:include filename="$(find openarm_description)/urdf/robot/${arm_type}.urdf.xacro" />
     <link name="base_link"/>
     <joint name="world_to_pedestal" type="fixed">
